File: Fuzz.brd (EAGLE design)
At the start: 160 x 100 mm, 19 parts, among them J1 DCJ0202, T1 2SC2509H, T2 2SC2509H

Commit message: Add files via upload
Other:
- board size 160 x 100 mm -> 152.4 x 100 mm
Changed lines of the file:
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@@
 <board>
 <plain>
-<wire x1="-8.89" y1="-1.27" x2="151.11" y2="-1.27" width="0" layer="20"/>
-<wire x1="151.11" y1="-1.27" x2="151.11" y2="98.73" width="0" layer="20"/>
-<wire x1="151.11" y1="98.73" x2="-8.89" y2="98.73" width="0" layer="20"/>
-<wire x1="-8.89" y1="98.73" x2="-8.89" y2="-1.27" width="0" layer="20"/>
+<wire x1="-11.43" y1="-1.27" x2="140.95" y2="-1.27" width="0" layer="20"/>
+<wire x1="140.95" y1="-1.27" x2="140.95" y2="98.73" width="0" layer="20"/>
+<wire x1="140.95" y1="98.73" x2="-11.43" y2="98.73" width="0" layer="20"/>
+<wire x1="-11.43" y1="98.73" x2="-11.43" y2="-1.27" width="0" layer="20"/>
 </plain>
 <attributes>
@@
 <wire x1="82.55" y1="13.97" x2="72.39" y2="24.13" width="1.27" layer="16"/>
 <wire x1="72.39" y1="24.13" x2="49.53" y2="24.13" width="1.27" layer="16"/>
-<wire x1="49.53" y1="24.13" x2="21.59" y2="52.07" width="0.762" layer="16"/>
+<wire x1="49.53" y1="24.13" x2="21.59" y2="52.07" width="1.27" layer="16"/>
 <wire x1="21.59" y1="52.07" x2="0.56" y2="52.07" width="1.27" layer="16"/>
 </signal>
@@
 <wire x1="123.19" y1="46.99" x2="117.89" y2="46.99" width="1.27" layer="1"/>
 <wire x1="117.89" y1="46.99" x2="93.76" y2="22.86" width="1.27" layer="1"/>
-<wire x1="34.29" y1="22.86" x2="24.13" y2="33.02" width="0.762" layer="1"/>
+<wire x1="34.29" y1="22.86" x2="24.13" y2="33.02" width="1.27" layer="1"/>
 <wire x1="93.76" y1="22.86" x2="34.29" y2="22.86" width="1.27" layer="1"/>
 <wire x1="0.46" y1="8.89" x2="0.46" y2="20.78" width="1.27" layer="16"/>
